File: trainlog.kicad_pcb (KiCad board)
At the start: 2 copper layers, 22 x 87.8 mm, 78 parts, among them J1 USB_C, J2 SD, J3 1PPS, Q1 AO3400A, Q2 AO3400A, SW1 SW_SPDT, U1 CP2102N-Axx-xQFN24, U2 USBLC6-4, U3 TP4056, U4 ESP32-WROOM-32U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

Commit message: updated gitignore
Parts:
- removed C24: 100n, otter:C_0402
- removed R25: 100k, otter:R_0402
- removed R26: 22k, otter:R_0402
- added R3: 540k, otter:R_0402, F.Cu at (90.2, 134.0)
- Q1, Q2: value AO3400A -> S8050
- R24: value 5k1 -> 120k
- U3: footprint Package_SO:Diodes_SO-8EP -> Package_SO:SSOP-8_3.95x5.21x3.27mm_P1.27mm
- U7: value SY8201 -> TLV62565DBVR; footprint Package_TO_SOT_SMD:SOT-23-6 -> Package_TO_SOT_SMD:SOT-23-5
- Y2: value Crystal -> 32.768kHz
- moved R30 25.0 mm to (95.6, 125.8), turned to 90 degrees
- moved R31 25.0 mm to (108.8, 104.6), turned to 180 degrees
- moved R24 5.52 mm to (90.8, 135.6), turned to 0 degrees
- moved R28 4.04 mm to (99.0, 130.0), turned to 0 degrees
- moved R29 3.75 mm to (99.6, 125.8), turned to -90 degrees
- moved C22 3.05 mm to (90.2, 138.6), turned to -90 degrees
- moved R23 3.03 mm to (91.2, 141.6), turned to 90 degrees
- moved C8 1.89 mm to (93.4, 141.4), turned to 0 degrees
- moved R1 0.63 mm to (97.7, 133.7), turned to -90 degrees
- moved C28 0.60 mm to (96.7, 125.8), turned to -90 degrees
- moved U7 0.57 mm to (92.8, 138.8), turned to 180 degrees
- moved Q2 0.36 mm to (98.5, 127.5), turned to 90 degrees
- moved Q1 0.27 mm to (96.8, 131.1)
Connections:
- L1 pad 1: Net-(C24-Pad2) -> Net-(L1-Pad1)
- Q1 pad 2: Net-(Q1-Pad2) -> DTR
- Q2 pad 1: Net-(Q1-Pad2) -> Net-(Q2-Pad1)
- Q2 pad 2: Net-(Q1-Pad1) -> RTS
- R24 pad 1: Net-(C22-Pad1) -> Net-(R3-Pad2)
- R24 pad 2: Net-(R24-Pad2) -> GND
- R28 pad 1: Net-(Q1-Pad1) -> Net-(Q2-Pad1)
- R28 pad 2: Net-(R28-Pad2) -> DTR
- R29 pad 1: Net-(Q1-Pad2) -> Net-(Q1-Pad1)
- R29 pad 2: Net-(R29-Pad2) -> RTS
- R30 pad 2: ESP_IO0 -> ESP_EN
- R31 pad 2: ESP_EN -> ESP_IO0
- U1 pad 19: Net-(R28-Pad2) -> RTS
- U1 pad 23: Net-(R29-Pad2) -> DTR
- U7 pad 1: Net-(C24-Pad1) -> Net-(C22-Pad1)
- U7 pad 3: Net-(R25-Pad2) -> Net-(L1-Pad1)
- U7 pad 4: Net-(R24-Pad2) -> Net-(C22-Pad1)
- U7 pad 5: Net-(C22-Pad1) -> Net-(R3-Pad2)
Routing:
- net Net-(Q1-Pad2): track 9.63 -> 0.00 mm, vias 2 -> 0
- net Net-(R25-Pad2): track 9.09 -> 0.00 mm, vias 2 -> 0
- net Net-(R3-Pad2): track 0.00 -> 7.53 mm
- net DTR: track 0.00 -> 6.94 mm, vias 0 -> 2
- net Net-(C24-Pad2): track 4.17 -> 0.00 mm
- net RTS: track 0.00 -> 3.54 mm
- net GND: track 33.1 -> 35.5 mm, vias 153 -> 156
- net ESP_EN: track 8.64 -> 6.41 mm
- net Net-(L1-Pad1): track 0.00 -> 1.97 mm
- net Net-(Q2-Pad1): track 0.00 -> 1.95 mm
- net Net-(Q1-Pad1): track 5.52 -> 7.43 mm
- net Net-(R28-Pad2): track 1.68 -> 0.00 mm
- net ESP_TXD: track 25.1 -> 23.5 mm
- net VBAT: track 103.3 -> 101.6 mm, vias 4 -> 5
- net Net-(R24-Pad2): track 1.60 -> 0.00 mm
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Other:
- board text added: "github.com/Jana-Marie/trainlog v1.1.0 by Jana Marie Hemsing Battery powered GPS, 9-DoF IMU & WiFi to SD & USB logger."
- board text removed: "github.com/Jana-Marie/trainlog v1.0.0 by Jana Marie Hemsing GPS, IMU & WiFi to SD & USB logger. This is part of an art project."
