File: trainlog.kicad_sch (KiCad schematic)
At the start: 78 parts, among them J1 USB_C, J2 SD, J3 1PPS, Q1 AO3400A, Q2 AO3400A, SW1 SW_SPDT, U1 CP2102N-Axx-xQFN24, U2 USBLC6-4, U3 TP4056, U4 ESP32-WROOM-32U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

Commit message: updated gitignore
Parts:
- removed C24: 100n, otter:C_0402, symbol Device:C_Small
- removed Q1, Q2: AO3400A, Package_TO_SOT_SMD:SOT-23, symbol Transistor_FET:2N7002
- removed R25: 100k, otter:R_0402, symbol Device:R_Small
- removed R26: 22k, otter:R_0402, symbol Device:R_Small
- removed U7: SY8201, Package_TO_SOT_SMD:SOT-23-6, symbol otter:JW5026
- added Q1, Q2: S8050, Package_TO_SOT_SMD:SOT-23, symbol Transistor_BJT:BC847
- added R3: 540k, otter:R_0402, symbol Device:R_Small
- added U7: TLV62565DBVR, Package_TO_SOT_SMD:SOT-23-5, symbol Regulator_Switching:TLV62568DBV
- R24: value 5k1 -> 120k
- Y2: value Crystal -> 32.768kHz
Connections:
- net +3V3: now also R3.1
- net ESP_EN: now also R30.2, Q2.3 (C); no longer R31.2
- net ESP_IO0: now also R31.2, Q1.3 (C); no longer R30.2
- net GND: now also R24.2, U7.2 (GND)
- net SD_CLK: now also J2.5 (CLK)
- net at C22.1, C8.1, R23.2: now also U7.1 (EN), U7.4 (VIN); no longer R24.1
- net at L1.1: now also U7.3 (SW)
- net at R28.1: now also Q2.1 (B)
- net DTR: now reaches R28.2
- net DTR: now also U1.23 (~{DTR}), Q1.2 (E); no longer U1.19 (~{RTS})
- net at R29.1: now also Q1.1 (B)
- net RTS: now reaches R29.2
- net RTS: now also U1.19 (~{RTS}), Q2.2 (E); no longer U1.23 (~{DTR})
- new net: R24.1, R3.2, U7.5 (FB)
Other:
- moved on the sheet: C22, C8, R23, R28, R29, R30, R31
